Commit message: 0529

File: dexmani_real/assets/robots/xhand/xarm7_xhand_right.urdf (robot description, URDF)
Before this commit: robot xarm7_xhand_right, 41 links, 40 joints
Links:
- added link calibration_mount, mass 0.025; collision cylinder length=0.005 radius=0.04; visual cylinder length=0.005 radius=0.04
- link flange_link: mass None -> 0.04
Joints:
- added joint calibration_mount_joint: type fixed, parent link_eef, child calibration_mount, origin xyz=0 0 0.0025 rpy=0 0 0
- joint flange_joint1: origin xyz=0 0 0.0 rpy=0 0 0 -> xyz=0 0 0.0025 rpy=0 0 0; parent link_eef -> calibration_mount
- joint flange_joint2: origin xyz=0.082 0 0.0436 rpy=3.1415926 0 0 -> xyz=0.0 0 0.043 rpy=0 -1.5708 0
