Commit message: 0701 retarget fix, but not fully tested

File: assets/robots/xhand/xarm7_xhand_right.urdf (robot description, URDF)
Before this commit: robot xarm7_xhand_right, 42 links, 41 joints
Joints:
- joint right_hand_thumb_rota_joint1: limit lower=-0.698 upper=1.57 effort=1.1 velocity=8.63 -> lower=-0.698 upper=1.745 effort=1.1 velocity=8.63
- joint right_hand_thumb_rota_joint2: limit lower=0 upper=1.57 effort=0.4 velocity=14.38 -> lower=0 upper=1.745 effort=0.4 velocity=14.38

File: assets/robots/xhand/xhand_right.urdf (robot description, URDF)
Before this commit: robot xhand_right, 30 links, 29 joints
Joints:
- joint right_hand_thumb_rota_joint1: limit lower=-0.698 upper=1.57 effort=1.1 velocity=8.63 -> lower=-0.698 upper=1.745 effort=1.1 velocity=8.63
- joint right_hand_thumb_rota_joint2: limit lower=0 upper=1.57 effort=0.4 velocity=14.38 -> lower=0 upper=1.745 effort=0.4 velocity=14.38

Commit message: 1028 temp

File: assets/robots/xhand/xarm7_xhand_right.urdf (robot description, URDF)
Before this commit: robot xarm7_xhand_right, 42 links, 41 joints
Links:
- removed link calibration_mount
- removed link flange_link
Joints:
- removed joint calibration_mount_joint
- removed joint flange_joint1
- joint flange_joint2: origin xyz=0.0 0 0.043 rpy=0 -1.5708 0 -> xyz=0.0 0 0.04 rpy=0 -1.5708 0; parent flange_link -> link_eef
- joint right_hand_mount_joint: origin xyz=-0.005 0 0.0 rpy=0 1.5708 0 -> xyz=-0.005 0 0 rpy=0 1.5707963267948966 0
